Commit message: feat #3 desciptionパッケージの整備

File: src/osp_naive/osp_description/urdf/osp.urdf (robot description, URDF)
Before this commit: robot osp_teleop, 5 links, 4 joints
Links:
- link base_link: geometry collision mesh filename=package://osp_description/meshes/base_link.STL; visual mesh filename=package://osp_description/meshes/base_link.STL
- link flipper_1: geometry collision mesh filename=package://osp_description/meshes/flipper_1.STL; visual mesh filename=package://osp_description/meshes/flipper_1.STL
- link flipper_2: geometry collision mesh filename=package://osp_description/meshes/flipper_2.STL; visual mesh filename=package://osp_description/meshes/flipper_2.STL
- link flipper_3: geometry collision mesh filename=package://osp_description/meshes/flipper_3.STL; visual mesh filename=package://osp_description/meshes/flipper_3.STL
- link flipper_4: geometry collision mesh filename=package://osp_description/meshes/flipper_4.STL; visual mesh filename=package://osp_description/meshes/flipper_4.STL
